File: ai03-pcb-guide.kicad_sch (KiCad schematic)
At the start: 15 parts, among them J1 Conn_01x04_Socket, U1 ATmega32U4-A, Y1 16MHz

Commit message: starting wiring tracks
Parts:
- added J2: AVR-ISP-6, random-keyboard-parts:Reset_Pretty-Mask, symbol Connector:AVR-ISP-6
Connections:
- net +5V: now also J2.2 (VCC)
- net Col 0: now also U1.29 (PB5); no longer U1.28 (PB4)
- net Col 1: now also U1.30 (PB6); no longer U1.29 (PB5)
- net Col 10: now also U1.21 (PD3); no longer U1.25 (PD4)
- net Col 11: now also U1.25 (PD4); no longer U1.26 (PD6)
- net Col 12: now also U1.26 (PD6); no longer U1.27 (PD7)
- net Col 13: now also U1.27 (PD7); no longer U1.9 (PB1)
- net Col 14: now also U1.28 (PB4); no longer U1.10 (PB2)
- net Col 2: now also U1.12 (PB7); no longer U1.30 (PB6)
- net Col 7: now also U1.11 (PB3), J2.1 (MISO); no longer U1.18 (PD0)
- net Col 8: now also U1.18 (PD0); no longer U1.19 (PD1)
- net Col 9: now also U1.19 (PD1); no longer U1.21 (PD3)
- net GND: now also J2.6 (GND)
- net RESET: now also J2.5 (~{RST})
- net Row 2: now also U1.38 (PF5); no longer U1.41 (PF0)
- net Row 3: now also U1.39 (PF4); no longer U1.40 (PF1)
- net Row 4: now also U1.40 (PF1); no longer U1.39 (PF4)
- net Row 5: now also U1.41 (PF0); no longer U1.38 (PF5)
- net DN: now reaches J1.2 (Pin_2), R2.2
- net DP: now reaches J1.3 (Pin_3), R3.1
- new net MOSI: J2.4 (MOSI), U1.10 (PB2)
- new net SCK: J2.3 (SCK), U1.9 (PB1)
- no-connect marks 5 -> 3
