File: ai03-pcb-guide.kicad_pcb (KiCad board)
At the start: 2 copper layers, 146 parts, among them SW1 SW_Push, SW10 8, SW11 9, SW12 0, SW13 - _, SW14 = +, SW15 \ |, SW17 Tab, SW18 Q, SW19 W, SW2 Esc, SW20 E, SW21 R, SW22 T, SW23 Y, SW24 U, SW25 I, SW26 O, SW27 P, SW28 { [, SW29 } ], SW3 1, SW30 Del, SW31 Ctrl, SW32 A, SW33 S, SW34 D, SW35 F, SW36 G, SW37 H, SW38 J, SW39 K, SW4 2, SW40 L, SW41 ; :, SW42 ' ", SW43 Return, SW44 Shift, SW45 Z, SW46 X, SW47 C, SW48 V, SW49 B, SW5 3, SW50 N, SW51 M, SW52 , <, SW53 . >, SW54 / ?, SW55 Shift, SW56 Fn, SW57 Option, SW58 Super, SW59 Space, SW6 4, SW60 Super, SW61 Option, SW62 Left Mouse, SW63 Middle Mouse, SW64 Right Mouse, SW7 5, SW8 6, SW9 7, U1 ATmega32U4-A, U2 PRTR5V0U2X, Y1 16MHz

Commit message: pcb finished except for routing
Parts:
- removed F1: 500m, Fuse:Fuse_1206_3216Metric
- removed R5, R6: 5.1k, Resistor_SMD:R_0805_2012Metric
- removed SW64: Right Mouse, Kalih Choc:KailhChoc-1.5U
- removed U2: PRTR5V0U2X, random-keyboard-parts:SOT143B
- removed USB1: HRO-TYPE-C-31-M-12, Type-C:HRO-TYPE-C-31-M-12
- added ?: , , F.Cu at (134.4, 94.7)
- added J1: Conn_01x04_Socket, Connector_Molex:Molex_Pico-EZmate_78171-0004_1x04-1MP_P1.20mm_Vertical, B.Cu at (53.6, 58.7)
- added Reset1: SW_Push, Button_Switch_SMD:SW_SPST_SKQG_WithStem, B.Cu at (135.2, 118.0)
- C8: footprint Diode_SMD:D_SOD-123 -> Resistor_SMD:R_0805_2012Metric
- R2: value 10k -> 22
- R4: value 22 -> 10k
- SW1: value SW_Push -> Esc; footprint Button_Switch_SMD:SW_SPST_SKQG_WithStem -> MX_Only:MXOnly-1U; moved to F.Cu
- SW10: value 8 -> 9
- SW11: value 9 -> 0
- SW12: value 0 -> - _
- SW13: value - _ -> = +
- SW14: value = + -> \ |
- SW15: value \ | -> ~
- SW16: value ~ -> Tab; footprint MX_Only:MXOnly-1U -> MX_Only:MXOnly-1.5U
- SW17: value Tab -> Q; footprint MX_Only:MXOnly-1.5U -> MX_Only:MXOnly-1U
- SW18: value Q -> W
- SW19: value W -> E
- SW2: value Esc -> 1
- SW20: value E -> R
- SW21: value R -> T
- SW22: value T -> Y
- SW23: value Y -> U
- SW24: value U -> I
- SW25: value I -> O
- SW26: value O -> P
- SW27: value P -> { [
- SW28: value { [ -> } ]
- SW29: value } ] -> Del; footprint MX_Only:MXOnly-1U -> MX_Only:MXOnly-1.5U
- SW3: value 1 -> 2
- SW30: value Del -> Ctrl; footprint MX_Only:MXOnly-1.5U -> MX_Only:MXOnly-1.75U
- SW31: value Ctrl -> A; footprint MX_Only:MXOnly-1.75U -> MX_Only:MXOnly-1U
- SW32: value A -> S
- SW33: value S -> D
- SW34: value D -> F
- SW35: value F -> G
- SW36: value G -> H
- SW37: value H -> J
- SW38: value J -> K
- SW39: value K -> L
- SW4: value 2 -> 3
- SW40: value L -> ; :
- SW41: value ; : -> ' "
- SW42: value ' " -> Return; footprint MX_Only:MXOnly-1U -> MX_Only:MXOnly-2.25U
- SW43: value Return -> Shift
- SW44: value Shift -> Z; footprint MX_Only:MXOnly-2.25U -> MX_Only:MXOnly-1U
- SW45: value Z -> X
- SW46: value X -> C
- SW47: value C -> V
- SW48: value V -> B
- SW49: value B -> N
- SW5: value 3 -> 4
- SW50: value N -> M
- SW51: value M -> , <
- SW52: value , < -> . >
- SW53: value . > -> / ?
- SW54: value / ? -> Shift; footprint MX_Only:MXOnly-1U -> MX_Only:MXOnly-1.75U
- SW55: value Shift -> Fn; footprint MX_Only:MXOnly-1.75U -> MX_Only:MXOnly-1U
- SW56: value Fn -> Option
- SW57: value Option -> Super; footprint MX_Only:MXOnly-1U -> MX_Only:MXOnly-1.5U
- SW58: value Super -> Space; footprint MX_Only:MXOnly-1.5U -> MX_Only:MXOnly-6U
- SW59: value Space -> Super; footprint MX_Only:MXOnly-6U -> MX_Only:MXOnly-1.5U
- SW6: value 4 -> 5
- SW60: value Super -> Option; footprint MX_Only:MXOnly-1.5U -> MX_Only:MXOnly-1U
- SW61: value Option -> Left Mouse; footprint MX_Only:MXOnly-1U -> Kalih Choc:KailhChoc-1.5U
- SW62: value Left Mouse -> Middle Mouse; footprint Kalih Choc:KailhChoc-1.5U -> Kalih Choc:KailhChoc-1U
- SW63: value Middle Mouse -> Right Mouse; footprint Kalih Choc:KailhChoc-1U -> Kalih Choc:KailhChoc-1.5U
- SW7: value 5 -> 6
- SW8: value 6 -> 7
- SW9: value 7 -> 8
- moved D55 259.1 mm to (287.1, 108.2), turned to 90 degrees
- moved D15 251.9 mm to (287.1, 51.1), turned to 90 degrees
- moved D29 249.8 mm to (282.3, 70.1), turned to 90 degrees
- moved D42 244.9 mm to (275.2, 89.2), turned to 90 degrees
- moved SW29 233.2 mm to (277.3, 66.1)
- moved D14 232.9 mm to (268.0, 51.1), turned to 90 degrees
- moved D54 232.8 mm to (260.9, 108.2), turned to 90 degrees
- moved D28 226.2 mm to (258.5, 70.1), turned to 90 degrees
- moved D41 214.3 mm to (244.2, 89.2), turned to 90 degrees
- moved D13 213.9 mm to (249.0, 51.1), turned to 90 degrees
- moved D60 212.0 mm to (239.5, 127.3), turned to 90 degrees
- moved D27 207.2 mm to (239.5, 70.1), turned to 90 degrees
- moved D53 206.5 mm to (234.7, 108.2), turned to 90 degrees
- moved D12 195.1 mm to (229.9, 51.1), turned to 90 degrees
- moved D40 195.1 mm to (225.2, 89.2), turned to 90 degrees
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Connections:
- R2 pad 1: GND -> D-
- R2 pad 2: Net-(U1-~{HWB}/PE2) -> Net-(J1-Pin_2)
- R3 pad 2: D- -> D+
- R4 pad 1: D+ -> GND
- R4 pad 2: Net-(U2-IO1) -> Net-(U1-~{HWB}/PE2)
- SW1 pad 1: GND -> Col 0
- SW1 pad 2: RESET -> Net-(D1-A)
- SW10 pad 1: Col 8 -> Col 9
- SW10 pad 2: Net-(D9-A) -> Net-(D10-A)
- SW11 pad 1: Col 9 -> Col 10
- SW11 pad 2: Net-(D10-A) -> Net-(D11-A)
- SW12 pad 1: Col 10 -> Col 11
- SW12 pad 2: Net-(D11-A) -> Net-(D12-A)
- SW13 pad 1: Col 11 -> Col 12
- SW13 pad 2: Net-(D12-A) -> Net-(D13-A)
- SW14 pad 1: Col 12 -> Col 13
- SW14 pad 2: Net-(D13-A) -> Net-(D14-A)
- SW15 pad 1: Col 13 -> Col 14
- SW15 pad 2: Net-(D14-A) -> Net-(D15-A)
- SW16 pad 1: Col 14 -> Col 0
- SW16 pad 2: Net-(D15-A) -> Net-(D16-A)
- SW17 pad 1: Col 0 -> Col 1
- SW17 pad 2: Net-(D16-A) -> Net-(D17-A)
- SW18 pad 1: Col 1 -> Col 2
- SW18 pad 2: Net-(D17-A) -> Net-(D18-A)
- SW19 pad 1: Col 2 -> Col 3
- SW19 pad 2: Net-(D18-A) -> Net-(D19-A)
- SW2 pad 1: Col 0 -> Col 1
- SW2 pad 2: Net-(D1-A) -> Net-(D2-A)
- SW20 pad 1: Col 3 -> Col 4
- SW20 pad 2: Net-(D19-A) -> Net-(D20-A)
- SW21 pad 1: Col 4 -> Col 5
- SW21 pad 2: Net-(D20-A) -> Net-(D21-A)
- SW22 pad 1: Col 5 -> Col 6
- SW22 pad 2: Net-(D21-A) -> Net-(D22-A)
- SW23 pad 1: Col 6 -> Col 7
- SW23 pad 2: Net-(D22-A) -> Net-(D23-A)
- SW24 pad 1: Col 7 -> Col 8
- SW24 pad 2: Net-(D23-A) -> Net-(D24-A)
- SW25 pad 1: Col 8 -> Col 9
- SW25 pad 2: Net-(D24-A) -> Net-(D25-A)
- SW26 pad 1: Col 9 -> Col 10
- SW26 pad 2: Net-(D25-A) -> Net-(D26-A)
- SW27 pad 1: Col 10 -> Col 11
- SW27 pad 2: Net-(D26-A) -> Net-(D27-A)
- SW28 pad 1: Col 11 -> Col 12
- SW28 pad 2: Net-(D27-A) -> Net-(D28-A)
- SW29 pad 1: Col 12 -> Col 14
- SW29 pad 2: Net-(D28-A) -> Net-(D29-A)
- SW3 pad 1: Col 1 -> Col 2
- SW3 pad 2: Net-(D2-A) -> Net-(D3-A)
- SW30 pad 1: Col 14 -> Col 0
- SW30 pad 2: Net-(D29-A) -> Net-(D30-A)
- SW31 pad 1: Col 0 -> Col 1
- SW31 pad 2: Net-(D30-A) -> Net-(D31-A)
- SW32 pad 1: Col 1 -> Col 2
- SW32 pad 2: Net-(D31-A) -> Net-(D32-A)
- SW33 pad 1: Col 2 -> Col 3
- SW33 pad 2: Net-(D32-A) -> Net-(D33-A)
- SW34 pad 1: Col 3 -> Col 4
- SW34 pad 2: Net-(D33-A) -> Net-(D34-A)
- SW35 pad 1: Col 4 -> Col 5
- SW35 pad 2: Net-(D34-A) -> Net-(D35-A)
- SW36 pad 1: Col 5 -> Col 6
- SW36 pad 2: Net-(D35-A) -> Net-(D36-A)
- SW37 pad 1: Col 6 -> Col 7
- SW37 pad 2: Net-(D36-A) -> Net-(D37-A)
- SW38 pad 1: Col 7 -> Col 8
- SW38 pad 2: Net-(D37-A) -> Net-(D38-A)
- SW39 pad 1: Col 8 -> Col 9
- SW39 pad 2: Net-(D38-A) -> Net-(D39-A)
- SW4 pad 1: Col 2 -> Col 3
- SW4 pad 2: Net-(D3-A) -> Net-(D4-A)
- SW40 pad 1: Col 9 -> Col 10
- SW40 pad 2: Net-(D39-A) -> Net-(D40-A)
- SW41 pad 1: Col 10 -> Col 11
- SW41 pad 2: Net-(D40-A) -> Net-(D41-A)
- SW42 pad 1: Col 11 -> Col 13
- SW42 pad 2: Net-(D41-A) -> Net-(D42-A)
- SW43 pad 1: Col 13 -> Col 0
- SW43 pad 2: Net-(D42-A) -> Net-(D43-A)
- SW44 pad 1: Col 0 -> Col 1
- SW44 pad 2: Net-(D43-A) -> Net-(D44-A)
- SW45 pad 1: Col 1 -> Col 2
- SW45 pad 2: Net-(D44-A) -> Net-(D45-A)
- SW46 pad 1: Col 2 -> Col 3
- SW46 pad 2: Net-(D45-A) -> Net-(D46-A)
- SW47 pad 1: Col 3 -> Col 4
- SW47 pad 2: Net-(D46-A) -> Net-(D47-A)
- SW48 pad 1: Col 4 -> Col 5
- SW48 pad 2: Net-(D47-A) -> Net-(D48-A)
- SW49 pad 1: Col 5 -> Col 6
- SW49 pad 2: Net-(D48-A) -> Net-(D49-A)
- SW5 pad 1: Col 3 -> Col 4
- SW5 pad 2: Net-(D4-A) -> Net-(D5-A)
- SW50 pad 1: Col 6 -> Col 7
- SW50 pad 2: Net-(D49-A) -> Net-(D50-A)
- SW51 pad 1: Col 7 -> Col 8
- SW51 pad 2: Net-(D50-A) -> Net-(D51-A)
- SW52 pad 1: Col 8 -> Col 9
- SW52 pad 2: Net-(D51-A) -> Net-(D52-A)
- SW53 pad 1: Col 9 -> Col 10
- SW53 pad 2: Net-(D52-A) -> Net-(D53-A)
- SW54 pad 1: Col 10 -> Col 12
- SW54 pad 2: Net-(D53-A) -> Net-(D54-A)
- SW55 pad 1: Col 12 -> Col 14
- SW55 pad 2: Net-(D54-A) -> Net-(D55-A)
- SW56 pad 1: Col 14 -> Col 0
- SW56 pad 2: Net-(D55-A) -> Net-(D56-A)
- SW57 pad 1: Col 0 -> Col 1
- SW57 pad 2: Net-(D56-A) -> Net-(D57-A)
- SW58 pad 1: Col 1 -> Col 5
- SW58 pad 2: Net-(D57-A) -> Net-(D58-A)
- SW59 pad 1: Col 5 -> Col 9
- SW59 pad 2: Net-(D58-A) -> Net-(D59-A)
- SW6 pad 1: Col 4 -> Col 5
- SW6 pad 2: Net-(D5-A) -> Net-(D6-A)
- SW60 pad 1: Col 9 -> Col 10
- SW60 pad 2: Net-(D59-A) -> Net-(D60-A)
- SW61 pad 1: Col 10 -> Col 4
- SW61 pad 2: Net-(D60-A) -> Net-(D61-A)
- SW62 pad 1: Col 4 -> Col 5
- SW62 pad 2: Net-(D61-A) -> Net-(D62-A)
- SW63 pad 1: Col 5 -> Col 6
- SW63 pad 2: Net-(D62-A) -> Net-(D63-A)
- SW7 pad 1: Col 5 -> Col 6
- SW7 pad 2: Net-(D6-A) -> Net-(D7-A)
- SW8 pad 1: Col 6 -> Col 7
- SW8 pad 2: Net-(D7-A) -> Net-(D8-A)
- SW9 pad 1: Col 7 -> Col 8
- SW9 pad 2: Net-(D8-A) -> Net-(D9-A)
Other:
- board outline added: 285.8 x 114.3 mm

Commit message: more revisions
Parts:
- removed the C7 at (107.9, 120.5)
- SW43: footprint MX_Only:MXOnly-2.25U -> MX_Only:MXOnly-2.25U-ReversedStabilizers-NoLED
- SW58: footprint MX_Only:MXOnly-6U -> MX_Only:MXOnly-6U-ReversedStabilizers-NoLED
- moved R3 0.39 mm to (115.8, 113.6)
- moved R2 0.33 mm to (113.7, 113.6)
- moved D3 0.33 mm to (58.3, 50.8)
- moved D16 0.33 mm to (24.9, 69.9)
- moved ? 0.33 mm to (134.1, 94.5)
- moved C1 0.33 mm to (132.5, 125.7)
- moved C2 0.33 mm to (132.5, 123.2)
- moved C3 0.33 mm to (119.0, 115.2)
- moved C4 0.33 mm to (108.2, 127.9)
- moved C5 0.33 mm to (120.3, 132.0)
- moved C6 0.33 mm to (125.2, 118.8)
- moved C7 0.33 mm to (109.8, 115.7)
- moved D1 0.33 mm to (20.2, 50.8)
- moved D10 0.33 mm to (191.6, 50.8)
- moved D11 0.33 mm to (210.7, 50.8)
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- renumbered C8 to C7
Other:
- board size 285.8 x 114.3 mm -> 284.4 x 97 mm

Commit message: fixing issues
Other:
- board size 284.4 x 97 mm -> 284.5 x 113.1 mm
