File: ai03-pcb-guide.kicad_pcb (KiCad board)
At the start: 2 copper layers, 284.5 x 113.1 mm, 142 parts, among them J1 Conn_01x04_Socket, SW1 Esc, SW10 9, SW11 0, SW12 - _, SW13 = +, SW14 \ |, SW16 Tab, SW17 Q, SW18 W, SW19 E, SW2 1, SW20 R, SW21 T, SW22 Y, SW23 U, SW24 I, SW25 O, SW26 P, SW27 { [, SW28 } ], SW29 Del, SW3 2, SW30 Ctrl, SW31 A, SW32 S, SW33 D, SW34 F, SW35 G, SW36 H, SW37 J, SW38 K, SW39 L, SW4 3, SW40 ; :, SW41 ' ", SW42 Return, SW43 Shift, SW44 Z, SW45 X, SW46 C, SW47 V, SW48 B, SW49 N, SW5 4, SW50 M, SW51 , <, SW52 . >, SW53 / ?, SW54 Shift, SW55 Fn, SW56 Option, SW57 Super, SW58 Space, SW59 Super, SW6 5, SW60 Option, SW61 Left Mouse, SW62 Middle Mouse, SW63 Right Mouse, SW7 6, SW8 7, SW9 8, U1 ATmega32U4-A, Y1 16MHz

Commit message: starting wiring tracks
Parts:
- added J2: AVR-ISP-6, random-keyboard-parts:Reset_Pretty-Mask, F.Cu at (87.1, 160.4)
Connections:
- net Net-(J1-Pin_2) renamed /DN
- net Net-(J1-Pin_3) renamed /DP
- U1 pad 10: Col 14 -> MOSI
- U1 pad 11: unconnected-(U1-PB3-Pad11) -> Col 7
- U1 pad 12: unconnected-(U1-PB7-Pad12) -> Col 2
- U1 pad 18: Col 7 -> Col 8
- U1 pad 19: Col 8 -> Col 9
- U1 pad 21: Col 9 -> Col 10
- U1 pad 25: Col 10 -> Col 11
- U1 pad 26: Col 11 -> Col 12
- U1 pad 27: Col 12 -> Col 13
- U1 pad 28: Col 0 -> Col 14
- U1 pad 29: Col 1 -> Col 0
- U1 pad 30: Col 2 -> Col 1
- U1 pad 38: Row 5 -> Row 2
- U1 pad 39: Row 4 -> Row 3
- U1 pad 40: Row 3 -> Row 4
- U1 pad 41: Row 2 -> Row 5
- U1 pad 9: Col 13 -> SCK
Routing:
- net Row 0: track 0.00 -> 284.1 mm
- net Row 1: track 0.00 -> 253.1 mm
- net Col 5: track 0.00 -> 113.0 mm
- net Col 6: track 0.00 -> 110.5 mm
- net Col 4: track 0.00 -> 105.5 mm
- net /DN: track 0.00 -> 102.5 mm
- net /DP: track 0.00 -> 101.4 mm
- net Col 0: track 0.00 -> 93.3 mm
- net Col 1: track 0.00 -> 90.1 mm
- net Col 10: track 0.00 -> 88.0 mm
- net Col 9: track 0.00 -> 86.1 mm
- net Col 7: track 0.00 -> 67.4 mm
- net Col 8: track 0.00 -> 67.0 mm
- net Col 3: track 0.00 -> 67.0 mm
- net Col 2: track 0.00 -> 67.0 mm
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
Commit message: more tracing work
Parts:
- moved R1 54.0 mm to (103.0, 165.0)
- moved Reset1 54.0 mm to (109.0, 165.1)
- moved C6 3.33 mm to (128.5, 119.0)
- moved C3 2.29 mm to (119.5, 113.0)
- moved C7 1.52 mm to (108.2, 115.8)
- moved C1 1.48 mm to (131.0, 125.7)
- moved C2 1.48 mm to (131.0, 123.2)
- moved Y1 0.93 mm to (127.3, 124.6), turned to 90 degrees
- moved R4 0.65 mm to (111.5, 131.8)
Connections:
- U1 pad 12: Col 2 -> Col 11
- U1 pad 25: Col 11 -> Col 12
- U1 pad 26: Col 12 -> Col 13
- U1 pad 27: Col 13 -> Col 14
- U1 pad 28: Col 14 -> Col 4
- U1 pad 31: Col 3 -> Col 2
- U1 pad 32: Col 4 -> Col 3
Routing:
- net Row 3: track 0.00 -> 249.9 mm
- net Row 2: track 0.00 -> 242.3 mm
- net Row 4: track 0.00 -> 202.5 mm
- net +5V: track 0.00 -> 199.9 mm, vias 0 -> 6
- net GND: track 0.00 -> 196.5 mm, vias 0 -> 7
- net Col 0: track 93.3 -> 157.7 mm
- net Row 5: track 0.00 -> 50.7 mm
- net Col 1: track 90.1 -> 135.5 mm
- net Col 2: track 67.0 -> 109.3 mm
- net Col 3: track 67.0 -> 96.6 mm
- net Col 4: track 105.5 -> 119.6 mm
- net Net-(D61-A): track 0.00 -> 10.4 mm
- net Net-(D63-A): track 0.00 -> 10.4 mm
- net Net-(D62-A): track 0.00 -> 10.4 mm
- net XTAL1: track 0.00 -> 9.36 mm
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- added copper zone on B.Cu, net GND
- added copper zone on F.Cu, net GND

Commit message: most wiring complete
Parts:
- moved J2 94.4 mm to (173.8, 123.0), turned to 180 degrees
- moved Reset1 70.6 mm to (165.6, 122.8)
- moved R1 69.2 mm to (159.2, 124.8), turned to 0 degrees
- moved C5 3.02 mm to (123.2, 131.5)
Connections:
- J2 pad 1: Col 7 -> Col 9
- U1 pad 1: Row 0 -> Row 3
- U1 pad 11: Col 7 -> Col 9
- U1 pad 12: Col 11 -> Col 10
- U1 pad 18: Col 8 -> Col 11
- U1 pad 19: Col 9 -> Col 12
- U1 pad 21: Col 10 -> Col 13
- U1 pad 25: Col 12 -> Col 14
- U1 pad 26: Col 13 -> Col 5
- U1 pad 27: Col 14 -> Col 6
- U1 pad 28: Col 4 -> Col 0
- U1 pad 29: Col 0 -> Col 1
- U1 pad 30: Col 1 -> Col 2
- U1 pad 31: Col 2 -> Col 3
- U1 pad 32: Col 3 -> Col 4
- U1 pad 36: Col 5 -> Row 5
- U1 pad 37: Row 1 -> Row 4
- U1 pad 38: Row 2 -> Row 0
- U1 pad 39: Row 3 -> Row 1
- U1 pad 40: Row 4 -> Row 2
- U1 pad 41: Row 5 -> Col 7
- U1 pad 8: Col 6 -> Col 8
Routing:
- net Col 14: track 62.0 -> 256.5 mm, vias 0 -> 1
- net Col 13: track 42.7 -> 236.6 mm, vias 0 -> 3
- net Col 11: track 44.0 -> 213.9 mm, vias 0 -> 1
- net Row 1: track 253.1 -> 414.5 mm, vias 0 -> 2
- net Col 12: track 62.1 -> 221.7 mm, vias 0 -> 1
- net Row 0: track 284.1 -> 440.7 mm
- net Row 2: track 242.3 -> 376.0 mm, vias 0 -> 2
- net Col 9: track 86.1 -> 211.7 mm, vias 0 -> 1
- net Col 10: track 88.0 -> 208.7 mm, vias 0 -> 1
- net RESET: track 0.00 -> 94.2 mm, vias 0 -> 4
- net Col 7: track 67.4 -> 158.0 mm, vias 0 -> 3
- net Col 8: track 67.0 -> 149.7 mm, vias 0 -> 3
- net SCK: track 0.00 -> 74.2 mm, vias 0 -> 1
- net MOSI: track 0.00 -> 73.2 mm, vias 0 -> 1
- net GND: track 196.5 -> 258.0 mm, vias 7 -> 10
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
Commit message: added trackpoint wiring
Parts:
- added C8: 2.2 uF, Capacitor_SMD:C_0805_2012Metric, B.Cu at (190.5, 93.7)
- added J3: Conn_01x05_Socket, Connector_Molex:Molex_Pico-EZmate_78171-0005_1x05-1MP_P1.20mm_Vertical, B.Cu at (181.8, 94.5)
- added R5: 100k, Resistor_SMD:R_0805_2012Metric, B.Cu at (187.3, 93.7)
- added R6: 4.7k, Resistor_SMD:R_0805_2012Metric, B.Cu at (187.3, 97.6)
- added R7: 4.7k, Resistor_SMD:R_0805_2012Metric, B.Cu at (190.5, 97.6)
- C7: footprint Resistor_SMD:R_0805_2012Metric -> Capacitor_SMD:C_0805_2012Metric
- J2: moved to B.Cu
- turned J2 to 0 degrees
Connections:
- U1 pad 20: unconnected-(U1-PD2-Pad20) -> D
- U1 pad 22: unconnected-(U1-PD5-Pad22) -> CLK
Routing:
- net D: track 0.00 -> 96.6 mm, vias 0 -> 4
- net +5V: track 252.3 -> 346.5 mm, vias 9 -> 13
- net CLK: track 0.00 -> 94.1 mm, vias 0 -> 4
- net GND: track 258.0 -> 343.0 mm, vias 10 -> 14
- net unconnected-(U1-PD5-Pad22): track 42.8 -> 0.00 mm, vias 3 -> 0
- net unconnected-(U1-PD2-Pad20): track 42.1 -> 0.00 mm, vias 3 -> 0
- net RST: track 0.00 -> 7.16 mm
- net Col 13: track 236.6 -> 235.0 mm
- net Row 2: track 376.0 -> 374.9 mm
