File: ai03-pcb-guide.kicad_pcb (KiCad board)
At the start: 2 copper layers, 284.5 x 113.1 mm, 148 parts, among them J1 Conn_01x04_Socket, J2 AVR-ISP-6, J3 Conn_01x05_Socket, SW1 Esc, SW10 9, SW11 0, SW12 - _, SW13 = +, SW14 \ |, SW16 Tab, SW17 Q, SW18 W, SW19 E, SW2 1, SW20 R, SW21 T, SW22 Y, SW23 U, SW24 I, SW25 O, SW26 P, SW27 { [, SW28 } ], SW29 Del, SW3 2, SW30 Ctrl, SW31 A, SW32 S, SW33 D, SW34 F, SW35 G, SW36 H, SW37 J, SW38 K, SW39 L, SW4 3, SW40 ; :, SW41 ' ", SW42 Return, SW43 Shift, SW44 Z, SW45 X, SW46 C, SW47 V, SW48 B, SW49 N, SW5 4, SW50 M, SW51 , <, SW52 . >, SW53 / ?, SW54 Shift, SW55 Fn, SW56 Option, SW57 Super, SW58 Space, SW59 Super, SW6 5, SW60 Option, SW61 Left Mouse, SW62 Middle Mouse, SW63 Right Mouse, SW7 6, SW8 7, SW9 8, U1 ATmega32U4-A, Y1 16MHz

Commit message: Almost finished
Parts:
- added G***: LOGO, LOGO, F.Cu at (134.1, 104.0)
- added REF**: MountingHole_2.2mm_M2, MountingHole:MountingHole_2.2mm_M2, F.Cu at (124.6, 94.0)
- added REF**: MountingHole_2.2mm_M2, MountingHole:MountingHole_2.2mm_M2, F.Cu at (143.6, 94.0)
- C1, C2, C3, C4, C5, C6, C7, C8: footprint Capacitor_SMD:C_0805_2012Metric -> Capacitor_SMD:C_0603_1608Metric
- R1, R2, R3, R4, R5, R6, R7: footprint Resistor_SMD:R_0805_2012Metric -> Resistor_SMD:R_0603_1608Metric
- moved D35 7.23 mm to (134.1, 83.2)
- moved C3 1.44 mm to (118.7, 114.2)
- moved ? 0.50 mm to (134.1, 94.0)
Routing:
- net +5V: track 346.5 -> 351.1 mm, vias 13 -> 15
- net Row 2: track 374.9 -> 379.4 mm
- net Col 7: track 158.0 -> 160.8 mm, vias 3 -> 5
- net Col 5: track 139.2 -> 141.2 mm
- net Col 6: track 162.6 -> 164.3 mm
- net Net-(U1-UCAP): track 6.63 -> 5.10 mm
- net GND: track 343.0 -> 344.6 mm
- net Net-(D35-A): track 8.48 -> 7.64 mm

Commit message: Rev 1.0
Connections:
- J3 pad 1: CLK -> GND
- J3 pad 2: +5V -> D
- J3 pad 3: GND -> CLK
- J3 pad 4: D -> RST
- J3 pad 5: RST -> +5V
Routing:
- net D: track 96.6 -> 91.6 mm
- net +5V: track 351.1 -> 355.9 mm, vias 15 -> 11
- net GND: track 344.6 -> 349.3 mm, vias 14 -> 16
- net CLK: track 94.1 -> 95.3 mm, vias 4 -> 6
Other:
- board text added: "Designed by Joseph Luken"
- board text added: "Tan63^{Rev 1.0}"

Commit message: routing tweaks
Routing:
- net Col 3: track 134.9 -> 136.8 mm
Changed lines of the file:
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@@
 	)
 	(segment
-		(start 83.83375 83.51625)
-		(end 83.83375 93.04125)
+		(start 106.613604 138.75)
+		(end 113.5 138.75)
 		(width 0.25)
 		(layer "F.Cu")
@@
 	)
 	(segment
-		(start 106.613604 138.75)
-		(end 113.5 138.75)
+		(start 101 128.25)
+		(end 101 133.136396)
 		(width 0.25)
 		(layer "F.Cu")
@@
 	)
 	(segment
-		(start 101 128.25)
-		(end 101 133.136396)
+		(start 82.70875 73.00875)
+		(end 77.94625 68.24625)
 		(width 0.25)
 		(layer "F.Cu")
@@
 	)
 	(segment
-		(start 78.5 63.895)
-		(end 78.5 78.1825)
+		(start 83.83375 96.33375)
+		(end 88.94125 101.44125)
 		(width 0.25)
 		(layer "F.Cu")
@@
 	)
 	(segment
-		(start 83.83375 93.04125)
+		(start 88.94125 101.44125)
 		(end 92.23375 101.44125)
 		(width 0.25)
@@
 	)
 	(segment
-		(start 114.5 139.75)
-		(end 116.25 139.75)
+		(start 83.83375 83.51625)
+		(end 83.83375 96.33375)
 		(width 0.25)
 		(layer "F.Cu")
@@
 	)
 	(segment
-		(start 78.5 78.1825)
-		(end 82.70875 82.39125)
+		(start 114.5 139.75)
+		(end 116.25 139.75)
 		(width 0.25)
 		(layer "F.Cu")
@@
 	)
 	(segment
+		(start 82.70875 82.39125)
+		(end 83.83375 83.51625)
+		(width 0.25)
+		(layer "F.Cu")
+		(net "Col 3")
+	)
+	(segment
 		(start 95.959188 126.3)
 		(end 99.05 126.3)
@@
 	(segment
 		(start 82.70875 82.39125)
-		(end 83.83375 83.51625)
+		(end 82.70875 73.00875)
 		(width 0.25)
 		(layer "F.Cu")
@@
 	)
 	(segment
-		(start 116.25 139.75)
-		(end 117.25 138.75)
+		(start 77.94625 68.24625)
+		(end 77.94625 63.34125)
 		(width 0.25)
 		(layer "F.Cu")
@@
 	)
 	(segment
-		(start 77.94625 63.34125)
-		(end 78.5 63.895)
+		(start 116.25 139.75)
+		(end 117.25 138.75)
 		(width 0.25)
 		(layer "F.Cu")
@@
 	)
 	(segment
+		(start 107.5 110.6)
+		(end 105.4 108.5)
+		(width 0.381)
+		(layer "F.Cu")
+		(net "GND")
+	)
+	(segment
 		(start 145.5 117.75)
 		(end 138.5 110.75)
@@
 	)
 	(segment
+		(start 105.4 108.5)
+		(end 105.4 107.7)
+		(width 0.381)
+		(layer "F.Cu")
+		(net "GND")
+	)
+	(segment
 		(start 152 120)
 		(end 150.321658 120)
@@
 	)
 	(segment
-		(start 132.5 110.75)
-		(end 131.5 109.75)
+		(start 107.5 111.25)
+		(end 107.5 110.6)
 		(width 0.381)
 		(layer "F.Cu")
@@
 	)
 	(segment
-		(start 107.75 105.25)
-		(end 107.5 105.5)
+		(start 105.4 107.7)
+		(end 107.75 105.35)
+		(width 0.381)
+		(layer "F.Cu")
+		(net "GND")
+	)
+	(segment
+		(start 132.5 110.75)
+		(end 131.5 109.75)
 		(width 0.381)
 		(layer "F.Cu")
@@
 	)
 	(segment
-		(start 107.5 105.5)
-		(end 107.5 111.25)
-		(width 0.381)
-		(layer "F.Cu")
-		(net "GND")
-	)
-	(segment
 		(start 158.9 93.4)
 		(end 162.9 97.4)
@@
 		(net "GND")
 	)
+	(segment
+		(start 107.75 105.35)
+		(end 107.75 105.25)
+		(width 0.381)
+		(layer "F.Cu")
+		(net "GND")
+	)
 	(via
 		(at 136.5 110.75)
@@
 	)
 	(segment
+		(start 53.88475 62.63475)
+		(end 53.88475 67.206408)
+		(width 0.381)
+		(layer "B.Cu")
+		(net "GND")
+	)
+	(segment
 		(start 117.925 112.525)
 		(end 117.925 114.2)
@@
 	)
 	(segment
-		(start 53.88475 60.25)
-		(end 53.88475 67.206408)
-		(width 0.381)
-		(layer "B.Cu")
-		(net "GND")
-	)
-	(segment
 		(start 120.68125 129.39375)
 		(end 122.09375 129.39375)
@@
 	)
 	(segment
-		(start 53.866 60.23125)
-		(end 53.88475 60.25)
-		(width 0.381)
-		(layer "B.Cu")
-		(net "GND")
-	)
-	(segment
 		(start 130.16875 121.45)
 		(end 130 121.45)
@@
 	)
 	(segment
+		(start 51.48125 60.23125)
+		(end 53.88475 62.63475)
+		(width 0.381)
+		(layer "B.Cu")
+		(net "GND")
+	)
+	(segment
 		(start 123.213078 121.949938)
 		(end 123.031766 122.13125)
@@
 		(width 0.381)
 		(layer "B.Cu")
-		(net "GND")
-	)
-	(segment
-		(start 51.48125 60.23125)
-		(end 53.866 60.23125)
-		(width 0.381)
-		(layer "B.Cu")

Commit message: rev1.0
Parts:
- moved D48 8.98 mm to (148.2, 107.9)
- moved D47 2.67 mm to (117.5, 108.3)
Routing:
- net GND: track 349.6 -> 386.8 mm, vias 16 -> 81
- net Net-(D48-A): track 8.48 -> 17.4 mm
- net Net-(D47-A): track 8.48 -> 7.79 mm
- net Col 5: track 141.2 -> 141.7 mm
