File: matrix.kicad_sch (KiCad schematic)
At the start: 126 parts, among them SW1 Esc, SW10 9, SW11 0, SW12 - _, SW13 = +, SW14 \ |, SW16 Tab, SW17 Q, SW18 W, SW19 E, SW2 1, SW20 R, SW21 T, SW22 Y, SW23 U, SW24 I, SW25 O, SW26 P, SW27 { [, SW28 } ], SW29 Del, SW3 2, SW30 Ctrl, SW31 A, SW32 S, SW33 D, SW34 F, SW35 G, SW36 H, SW37 J, SW38 K, SW39 L, SW4 3, SW40 ; :, SW41 ' ", SW42 Return, SW43 Shift, SW44 Z, SW45 X, SW46 C, SW47 V, SW48 B, SW49 N, SW5 4, SW50 M, SW51 , <, SW52 . >, SW53 / ?, SW54 Shift, SW55 Fn, SW56 Option, SW57 Super, SW58 Space, SW59 Super, SW6 5, SW60 Option, SW61 Left Mouse, SW62 Middle Mouse, SW63 Right Mouse, SW7 6, SW8 7, SW9 8

Commit message: Added LCSC Part # Field
Parts:
- D1, D10, D11, D12, D13, D14, D15, D16, D17, D18, D19, D2, D20, D21, D22, D23, D24, D25, D26, D27, D28, D29, D3, D30, D31, D32, D33, D34, D35, D36, D37, D38, D39, D4, D40, D41, D42, D43, D44, D45, D46, D47, D48, D49, D5, D50, D51, D52, D53, D54, D55, D56, D57, D58, D59, D6, D60, D61, D62, D63, D7, D8, D9: LCSC Part # (none) -> C83528
